Commit message: Remove Jittering, Wrist Camera Adjustion, Speed up Rendering

File: assets/automate/urdf/automate_franka.urdf (robot description, URDF)
Before this commit: robot panda, 12 links, 11 joints
Links:
- added link panda_camera, mass 1e-6; collision box size=0.0001 0.0001 0.0001; visual box size=0.02 0.02 0.02
Joints:
- added joint panda_camera_joint: type fixed, parent panda_hand, child panda_camera, origin xyz=0.08 0.0 0.03 rpy=0 0 0
